File: BusBoard.kicad_pcb (KiCad board)
At the start: 4 copper layers, 117.4 x 100 mm, 35 parts, among them J201 Conn_02x10_Row_Letter_First, J301 Conn_02x10_Row_Letter_First, J401 Conn_02x10_Row_Letter_First, J501 Conn_02x10_Row_Letter_First, J601 Conn_02x10_Row_Letter_First, J701 Conn_02x10_Row_Letter_First, U101 USBLC6-2SC6, U102 FE1.1s, U103 USBLC6-2SC6, U104 USBLC6-2SC6, U105 USBLC6-2SC6, U106 USBLC6-2SC6, Y101 12MHz

Commit message: chore: migrate <<HASH>> placeholder to <<VERSION>>
Aligns the KiCad title-block placeholder with the new versioning concept
documented at oe5xrx.org/docs/remote-station/hardware/versioning/.

The placeholder is substituted at CI time:
- Release build:  v1.5 → "1.5" (semver only, no `v`, no SHA)
- Debug build:    "BETA-<short-commit>"

No electrical or layout change — pure text replacement on the title-block
silkscreen text. Requires HW-Module-CI feat/version-placeholder
(OE5XRX/HW-Module-CI#4) to be merged first; otherwise CI substitutes
the old <<HASH>> token and leaves the new <<VERSION>> string literal
in the title block until the CI side catches up.

Co-Authored-By: Claude Opus 4.7 <noreply@anthropic.com>
Other:
- board text added: "<<VERSION>>"
- board text removed: "<<HASH>>"
Changed lines of the file:
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@@
 		)
 	)
-	(gr_text "<<HASH>>"
+	(gr_text "<<VERSION>>"
 		(at 80.905 107.692 0)
 		(layer "F.SilkS")
